Commit message: first commit

File: src/m2wr_description/urdf/rover.xacro (robot description, xacro)
@@ -28,12 +28,27 @@
     <material>Gazebo/Orange</material>
   </gazebo>
-  <gazebo reference="link_left_wheel">
+  <gazebo reference="link_back_left_wheel">
     <material>Gazebo/Blue</material>
   </gazebo>
-  <gazebo reference="link_right_wheel">
+  <gazebo reference="link_back_right_wheel">
     <material>Gazebo/Blue</material>
+  </gazebo>
+  <gazebo reference="link_front_left_wheel">
+    <material>Gazebo/Blue</material>
+  </gazebo>
+  <gazebo reference="link_front_right_wheel">
+    <material>Gazebo/Blue</material>
+  </gazebo>
+  <gazebo reference="link_front_left_hinge">
+    <material>Gazebo/Orange</material>
+  </gazebo>
+  <gazebo reference="link_front_right_hinge">
+    <material>Gazebo/Orange</material>
   </gazebo>
   <gazebo reference="camera_link">
     <material>Gazebo/Black</material>
+  </gazebo>
+  <gazebo reference="imu_link">
+    <material>Gazebo/white</material>
   </gazebo>
   <!-- camera -->
@@ -42,8 +57,8 @@
       <update_rate>30.0</update_rate>
       <camera name="head">
-        <horizontal_fov>1.3962634</horizontal_fov>
+        <horizontal_fov>1.777778</horizontal_fov>
         <image>
-          <width>800</width>
-          <height>800</height>
+          <width>960</width>
+          <height>616</height>
           <format>R8G8B8</format>
         </image>
@@ -77,16 +92,17 @@
     </sensor>
   </gazebo>
+  <!-- chassis -->
   <link name="link_chassis">
     <!-- pose and inertial -->
-    <pose>0 0 0.1 0 0 0</pose>
-    <inertial>
-      <mass value="2"/>
+    <pose>0 0 0 0 0 0</pose>
+    <inertial>
+      <mass value="0.796"/>
       <origin rpy="0 0 0" xyz="0 0 0"/>
-      <inertia ixx="0.001933" ixy="0" ixz="0" iyy="0.003533" iyz="0" izz="0.004933"/>
+      <inertia ixx="0.001573" ixy="0" ixz="0" iyy="0.004227" iyz="0" izz="0.005638"/>
     </inertial>
     <!-- body -->
     <collision name="collision_chassis">
       <geometry>
-        <box size="0.14 0.1 0.04"/>
+        <box size="0.25 0.15 0.035"/>
       </geometry>
     </collision>
@@ -94,158 +110,153 @@
       <origin rpy="0 0 0" xyz="0 0 0"/>
       <geometry>
-        <box size="0.14 0.1 0.04"/>
+        <box size="0.25 0.15 0.035"/>
       </geometry>
       <material name="blue"/>
     </visual>
-    <!-- front cylinder that holds the caster-->
-    <collision name="f_caster_wheel_hold">
-     <origin rpy=" 0 0 0" xyz="0.065 0 -0.025"/>
-      <geometry>
-        <cylinder length="0.0075" radius="0.0025"/>
-      </geometry>
-      <surface>
-        <friction>
-          <ode>
-            <mu>0</mu>
-            <mu2>0</mu2>
-            <slip1>0.0</slip1>
-            <slip2>0.0</slip2>
-          </ode>
-        </friction>
-      </surface>
-    </collision>
-    <visual>
-      <origin rpy="0 0 0" xyz="0.065 0 -0.025"/>
-      <geometry>
-        <cylinder length="0.0075" radius="0.0025"/>
-      </geometry>
-      <material name="blue"/>
-    </visual>
-    <!-- rear cylinder that holds the caster-->
-    <collision name="r_caster_wheel_hold">
-     <origin rpy=" 0 0 0" xyz="-0.065 0 -0.025"/>
-      <geometry>
-        <cylinder length="0.0075" radius="0.0025"/>
-      </geometry>
-      <surface>
-        <friction>
-          <ode>
-            <mu>0</mu>
-            <mu2>0</mu2>
-            <slip1>0.0</slip1>
-            <slip2>0.0</slip2>
-          </ode>
-        </friction>
-      </surface>
-    </collision>
-    <visual>
-      <origin rpy="0 0 0" xyz="-0.065 0 -0.025"/>
-      <geometry>
-        <cylinder length="0.0075" radius="0.0025"/>
-      </geometry>
-      <material name="blue"/>
-    </visual>
-    <!-- caster front -->
-    <collision name="caster_front_collision">
-      <origin rpy=" 0 0 0" xyz="0.065 0 -0.0275"/>
-      <geometry>
-        <sphere radius="0.00025"/>
-      </geometry>
-      <surface>
-        <friction>
-          <ode>
-            <mu>0</mu>
-            <mu2>0</mu2>
-            <slip1>0.0</slip1>
-            <slip2>0.0</slip2>
-          </ode>
-        </friction>
-      </surface>
-    </collision>
-    <visual name="caster_front_visual">
-      <origin rpy=" 0 0 0" xyz="0.065 0 -0.0275"/>
-      <geometry>
-        <sphere radius="0.00025"/>
-      </geometry>
-    </visual>
-    <!-- caster rear -->
-    <collision name="caster_rear_collision">
-      <origin rpy=" 0 0 0" xyz="-0.065 0.0 -0.0275"/>
-      <geometry>
-        <sphere radius="0.00025"/>
-      </geometry>
-      <surface>
-        <friction>
-          <ode>
-            <mu>0</mu>
-            <mu2>0</mu2>
-            <slip1>0.0</slip1>
-            <slip2>0.0</slip2>
-          </ode>
-        </friction>
-      </surface>
-    </collision>
-    <visual name="caster_rear_visual">
-      <origin rpy=" 0 0 0" xyz="-0.065 0.0 -0.0275"/>
-      <geometry>
-        <sphere radius="0.00025"/>
-      </geometry>
-    </visual>
-  </link>
-  <link name="link_right_wheel">
-    <inertial>
-      <mass value="0.5"/>
-      <origin rpy="0 1.5707 1.5707" xyz="0 0 0"/>
-      <inertia ixx="0.00012917" ixy="0" ixz="0" iyy="0.00012917" iyz="0" izz="0.000225"/>
-    </inertial>
-    <collision name="link_right_wheel_collision">
-      <origin rpy="0 1.5707 1.5707" xyz="0 0 0"/>
-      <geometry>
-        <cylinder length="0.015" radius="0.03"/>
-      </geometry>
-    </collision>
-    <visual name="link_right_wheel_visual">
-      <origin rpy="0 1.5707 1.5707" xyz="0 0 0"/>
-      <geometry>
-        <cylinder length="0.015" radius="0.03"/>
-      </geometry>
-    </visual>
-  </link>
-  <joint name="joint_right_wheel" type="continuous">
-    <origin rpy="0 0 0" xyz="0.01 -0.0575 0.0"/>
-    <child link="link_right_wheel"/>
-    <parent link="link_chassis"/>
+  </link>
+<!-- wheels & hinges -->
+<!-- Front right -->
+  <link name="link_front_right_wheel">
+    <inertial>
+      <mass value="0.049"/>
+      <origin rpy="0 1.5707 1.5707" xyz="0 0 0"/>
+      <inertia ixx="1.755e-5" ixy="0" ixz="0" iyy="1.755e-5" iyz="0" izz="3.001e-5"/>
+    </inertial>
+    <collision name="link_front_right_wheel_collision">
+      <origin rpy="0  -1.5707  -1.5707" xyz="0 0 0"/>
+      <geometry>
+        <cylinder length="0.025" radius="0.035"/>
+      </geometry>
+    </collision>
+    <visual name="link_front_right_wheel_visual">
+      <origin rpy="0  -1.5707  -1.5707" xyz="0 0 0"/>
+      <geometry>
+        <cylinder length="0.025" radius="0.035"/>
+      </geometry>
+    </visual>
+  </link>
+  <link name="link_front_right_hinge">
+    <inertial>
+      <mass value="1e-5"/>
+      <origin rpy="0 0 0" xyz="0 0 0"/>
+      <inertia ixx="1e-6" ixy="0" ixz="0" iyy="1e-6" iyz="0" izz="1e-6"/>
+    </inertial>
+  </link>
+  <joint name="joint_front_right_wheel" type="continuous">
+    <origin rpy="0 0 0" xyz="0 -0.015 0"/>
+    <child link="link_front_right_wheel"/>
+    <parent link="link_front_right_hinge"/>
     <axis rpy="0 0 0" xyz="0 1 0"/>
     <limit effort="5" velocity="10"/>
     <joint_properties damping="0.0" friction="0.0"/>
   </joint>
-  <link name="link_left_wheel">
-    <inertial>
-      <mass value="0.5"/>
-      <origin rpy="0 1.5707 1.5707" xyz="0 0 0"/>
-      <inertia ixx="0.00012917" ixy="0" ixz="0" iyy="0.00012917" iyz="0" izz="0.000225"/>
-    </inertial>
-    <collision name="link_left_wheel_collision">
-      <origin rpy="0 1.5707 1.5707" xyz="0 0 0"/>
-      <geometry>
-        <cylinder length="0.015" radius="0.03"/>
-      </geometry>
-    </collision>
-    <visual name="link_left_wheel_visual">
-      <origin rpy="0 1.5707 1.5707" xyz="0 0 0"/>
-      <geometry>
-        <cylinder length="0.015" radius="0.03"/>
-      </geometry>
-    </visual>
-  </link>
-  <joint name="joint_left_wheel" type="continuous">
-    <origin rpy="0 0 0" xyz="0.01 0.0575 0.0"/>
-    <child link="link_left_wheel"/>
-    <parent link="link_chassis"/>
+  <joint name="joint_front_right_hinge" type="revolute">
+    <origin rpy="0 0 0" xyz="0.125 -0.085 0.0"/>
+    <child link="link_front_right_hinge"/>
+    <parent link="link_chassis"/>
+    <axis rpy="0 0 0" xyz="0 0 1"/>
+    <limit  effort="10" velocity="5" lower="-0.610" upper="0.523"/>
+    <joint_properties damping="0.0" friction="0.0"/>
+  </joint>
+<!-- front left -->
+  <link name="link_front_left_wheel">
+    <inertial>
+      <mass value="0.049"/>
+      <origin rpy="0 1.5707 1.5707" xyz="0 0 0"/>
+      <inertia ixx="1.755e-5" ixy="0" ixz="0" iyy="1.755e-5" iyz="0" izz="3.001e-5"/>
+    </inertial>
+    <collision name="link_front_left_wheel_collision">
+      <origin rpy="0 1.5707 1.5707" xyz="0 0 0"/>
+      <geometry>
+        <cylinder length="0.025" radius="0.035"/>
+      </geometry>
+    </collision>
+    <visual name="link_front_left_wheel_visual">
+      <origin rpy="0 1.5707 1.5707" xyz="0 0 0"/>
+      <geometry>
+        <cylinder length="0.025" radius="0.035"/>
+      </geometry>
+    </visual>
+  </link>
+  <link name="link_front_left_hinge">
+    <inertial>
+      <mass value="1e-5"/>
+      <origin rpy="0 0 0" xyz="0 0 0"/>
+      <inertia ixx="1e-6" ixy="0" ixz="0" iyy="1e-6" iyz="0" izz="1e-6"/>
+    </inertial>
+  </link>
+  <joint name="joint_front_left_wheel" type="continuous">
+    <origin rpy="0 0 0" xyz="0.0 0.015 0.0"/>
+    <child link="link_front_left_wheel"/>
+    <parent link="link_front_left_hinge"/>
     <axis rpy="0 0 0" xyz="0 1 0"/>
     <limit effort="5" velocity="10"/>
     <joint_properties damping="0.0" friction="0.0"/>
   </joint>
-  <!-- Camera -->
+  <joint name="joint_front_left_hinge" type="revolute">
+    <origin rpy="0 0 0" xyz="0.125 0.085 0.0"/>
+    <child link="link_front_left_hinge"/>
+    <parent link="link_chassis"/>
+    <axis rpy="0 0 0" xyz="0 0 1"/>
+    <limit effort="10" velocity="5" lower= "-0.610" upper="0.523"/>
+    <joint_properties damping="0.0" friction="0.0"/>
+  </joint>
+<!-- back right -->
+  <link name="link_back_right_wheel">
+    <inertial>
+      <mass value="0.049"/>
+      <origin rpy="0 -1.5707 -1.5707" xyz="0 0 0"/>
+      <inertia ixx="1.755e-5" ixy="0" ixz="0" iyy="1.755e-5" iyz="0" izz="3.001e-5"/>
+    </inertial>
+    <collision name="link_back_right_wheel_collision">
+      <origin rpy="0 -1.5707 -1.5707" xyz="0 0 0"/>
+      <geometry>
+        <cylinder length="0.025" radius="0.035"/>
+      </geometry>
+    </collision>
+    <visual name="link_back_right_wheel_visual">
+      <origin rpy="0 -1.5707 -1.5707" xyz="0 0 0"/>
+      <geometry>
+        <cylinder length="0.025" radius="0.035"/>
+      </geometry>
+    </visual>
+  </link>
+  <joint name="joint_back_right_wheel" type="continuous">
+    <origin rpy="0 0 0" xyz="-0.125 -0.085  0"/>
+    <child link="link_back_right_wheel"/>
+    <parent link="link_chassis"/>
+    <axis rpy="0 0 0" xyz="0 1 0"/>
+    <limit effort="5" velocity="10"/>
+    <joint_properties damping="0.0" friction="0.0"/>
+  </joint>
+<!-- back left -->
+  <link name="link_back_left_wheel">
+    <inertial>
+      <mass value="0.049"/>
+      <origin rpy="0 1.5707 1.5707" xyz="0 0 0"/>
+      <inertia ixx="1.755e-5" ixy="0" ixz="0" iyy="1.755e-5" iyz="0" izz="3.001e-5"/>
+    </inertial>
+    <collision name="link_back_left_wheel_collision">
+      <origin rpy="0 1.5707 1.5707" xyz="0 0 0"/>
+      <geometry>
+        <cylinder length="0.025" radius="0.035"/>
+      </geometry>
+    </collision>
+    <visual name="link_back_left_wheel_visual">
+      <origin rpy="0 1.5707 1.5707" xyz="0 0 0"/>
+      <geometry>
+        <cylinder length="0.025" radius="0.035"/>
+      </geometry>
+    </visual>
+  </link>
+  <joint name="joint_back_left_wheel" type="continuous">
+    <origin rpy="0 0 0" xyz="-0.125 0.085 0.0"/>
+    <child link="link_back_left_wheel"/>
+    <parent link="link_chassis"/>
+    <axis rpy="0 0 0" xyz="0 1 0"/>
+    <limit effort="5" velocity="10"/>
+    <joint_properties damping="0.0" friction="0.0"/>
+  </joint>
+  <!-- Camera link & joint -->
   <link name="camera_link">
 	<inertial>
@@ -260,5 +271,5 @@
       	</geometry>
     </collision>
-    <visual name = "camera_link_visual">
+    <visual>
       	<origin xyz="0 0 0" rpy="0 0 0"/>
       	<geometry>
@@ -268,26 +279,92 @@
   </link>
   <joint name="camera_joint" type="fixed">
-	    <origin xyz="0.085 0 0.05" rpy="0 1.0466 0"/>
-	    <child link="camera_link"/>
-	    <parent link="link_chassis"/>
-            <axis rpy = "0 0 0" xyz="0 1 0" />
-  </joint>
-  <transmission name = "joint_left_wheel_trans">
+	<origin xyz="0.07 0 0.11" rpy="0 0.6266 0"/>
+	<child link="camera_link"/>
+	<parent link="link_chassis"/>
+	<axis rpy = "0 0 0" xyz="0 1 0" />
+  </joint>
+  <!--imu link and joint-->
+<link name="imu_link">
+  <inertial>
+    <mass value="1e-5"/>
+    <origin rpy="0 0 0" xyz="0 0 0"/>
+    <inertia ixx="1e-6" ixy="0" ixz="0" iyy="1e-6" iyz="0" izz="1e-6"/>
+  </inertial>
+  <visual>
+    <origin rpy="0 0 0" xyz="0 0 0"/>
+    <geometry>
+      <box size="0.01 0.01 0.01"/>
+    </geometry>
+  </visual>
+  <collision>
+    <origin rpy="0 0 0" xyz="0 0 0"/>
+    <geometry>
+      <box size="0.01 0.01 0.01"/>
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
Commit message: initial package

File: src/m2wr_description/urdf/rover.xacro (robot description, xacro)
@@ -48,8 +48,5 @@
   <gazebo reference="camera_link">
     <material>Gazebo/Black</material>
-  </gazebo>
-  <gazebo reference="imu_link">
-    <material>Gazebo/white</material>
-  </gazebo>
+	</gazebo>
   <!-- camera -->
   <gazebo reference="camera_link">
@@ -151,10 +148,10 @@
     <joint_properties damping="0.0" friction="0.0"/>
   </joint>
-  <joint name="joint_front_right_hinge" type="revolute">
+ <joint name="joint_front_right_hinge" type="revolute">
     <origin rpy="0 0 0" xyz="0.125 -0.085 0.0"/>
     <child link="link_front_right_hinge"/>
     <parent link="link_chassis"/>
     <axis rpy="0 0 0" xyz="0 0 1"/>
-    <limit  effort="10" velocity="5" lower="-0.610" upper="0.523"/>
+    <limit  effort="10" velocity="5" lower="-0.261" upper="0.174"/>
     <joint_properties damping="0.0" friction="0.0"/>
   </joint>
@@ -199,5 +196,5 @@
     <parent link="link_chassis"/>
     <axis rpy="0 0 0" xyz="0 0 1"/>
-    <limit effort="10" velocity="5" lower= "-0.610" upper="0.523"/>
+    <limit effort="10" velocity="5" lower= "-0.261" upper="0.174"/>
     <joint_properties damping="0.0" friction="0.0"/>
   </joint>
@@ -284,6 +281,10 @@
 	<axis rpy = "0 0 0" xyz="0 1 0" />
   </joint>
-  <!--imu link and joint-->
-<link name="imu_link">
+  <!-- IMU colour -->
+<!--<gazebo reference="imu_link">
+    <material>Gazebo/white</material>
+  </gazebo>-->
+<!--imu link and joint-->
+<!--<link name="imu_link">
   <inertial>
     <mass value="1e-5"/>
@@ -309,15 +310,15 @@
     <child link="imu_link"/>
     <axis rpy = "0 0 0" xyz="0 1 0"/>
-  </joint>
+  </joint>-->
+  <!--imu plugin-->
   <!--<gazebo reference="imu_link">
-    <gravity>true</gravity>
     <sensor name="imu_sensor" type="imu">
       <always_on>true</always_on>
-      <update_rate>100</update_rate>
+      <update_rate>100.0</update_rate>
       <visualize>true</visualize>
-      <topic>__default_topic__</topic>
+      <topic>imu_raw</topic>
       <plugin filename="libgazebo_ros_imu_sensor.so" name="imu_plugin">
-        <topicName>imu</topicName>
-        <bodyName>imu_link</bodyName>
+        <topicName>imu/data</topicName>
+        <bodyName>imu_body</bodyName>
         <updateRateHZ>10.0</updateRateHZ>
         <gaussianNoise>0.0</gaussianNoise>
@@ -327,5 +328,4 @@
         <initialOrientationAsReference>false</initialOrientationAsReference>
       </plugin>
-      <pose>0 0 0 0 0 0</pose>
     </sensor>
   </gazebo-->

Commit message: XACRO file update with IMU plugin and IMU sensor

File: src/m2wr_description/urdf/rover.xacro (robot description, xacro)
@@ -89,4 +89,25 @@
     </sensor>
   </gazebo>
+<!--imu plugin-->
+<gazebo reference="imu_link">
+<gravity>true</gravity>
+<sensor name="imu_sensor" type="imu">
+<always_on>true</always_on>
+<update_rate>100</update_rate>
+<visualize>true</visualize>
+<topic>__default_topic__</topic>
+<plugin filename="libgazebo_ros_imu_sensor.so" name="imu_plugin">
+<topicName>imu</topicName>
+<bodyName>imu_link</bodyName>
+<updateRateHZ>10.0</updateRateHZ>
+<gaussianNoise>0.0</gaussianNoise>
+<xyzOffset>0 0 0</xyzOffset>
+<rpyOffset>0 0 0</rpyOffset>
+<frameName>imu_link</frameName>
+<initialOrientationAsReference>false</initialOrientationAsReference>
+</plugin>
+<pose>0 0 0 0 0 0</pose>
+</sensor>
+</gazebo>
   <!-- chassis -->
   <link name="link_chassis">
@@ -281,4 +302,29 @@
 	<axis rpy = "0 0 0" xyz="0 1 0" />
   </joint>
+<link name="imu_link">
+<inertial>
+<mass value = "1e-5"/>
+<origin xyz="0 0 0" rpy="0 0 0"/>
+<inertia ixx="1e-6" ixy="0" ixz="0" iyy="1e-6" iyz="0" izz="1e-6" />
+</inertial>
+<collision name = "imu_link_collision">
+<origin xyz="0 0 0" rpy="0 0 0"/>
+<geometry>
+<box size="0.01 0.01 0.01"/>
+</geometry>
+</collision>
+<visual name = "imu_link_visual">
+<origin xyz="0 0 0" rpy="0 0 0"/>
+<geometry>
+<box size="0.01 0.01 0.01"/>
+</geometry>
+</visual>
+</link>
+<joint name="imu_joint" type="fixed">
+<origin xyz="0.0 0 0.05" rpy="0 0 0"/>
+<child link="imu_link"/>
+<parent link="link_chassis"/>
+<axis rpy = "0 0 0" xyz="0 1 0" />
+</joint>
   <!-- IMU colour -->
 <!--<gazebo reference="imu_link">

Commit message: 13/04/2021 commit

File: src/m2wr_description/urdf/rover.xacro (robot description, xacro)
@@ -174,5 +174,5 @@
     <parent link="link_chassis"/>
     <axis rpy="0 0 0" xyz="0 0 1"/>
-    <limit  effort="10" velocity="5" lower="-0.261" upper="0.174"/>
+    <limit  effort="5" velocity="5" lower="-0.43" upper="0.33"/>
     <joint_properties damping="0.0" friction="0.0"/>
   </joint>
@@ -217,5 +217,5 @@
     <parent link="link_chassis"/>
     <axis rpy="0 0 0" xyz="0 0 1"/>
-    <limit effort="10" velocity="5" lower= "-0.261" upper="0.174"/>
+    <limit effort="5" velocity="5" lower= "-0.33" upper="0.44"/>
     <joint_properties damping="0.0" friction="0.0"/>
   </joint>
@@ -297,5 +297,5 @@
   </link>
   <joint name="camera_joint" type="fixed">
-	<origin xyz="0.07 0 0.11" rpy="0 0.6266 0"/>
+	<origin xyz="0.07 0 0.11" rpy="0 0.5 0"/>
 	<child link="camera_link"/>
 	<parent link="link_chassis"/>
@@ -327,53 +327,4 @@
 <axis rpy = "0 0 0" xyz="0 1 0" />
 </joint>
-  <!-- IMU colour -->
-<!--<gazebo reference="imu_link">
-    <material>Gazebo/white</material>
-  </gazebo>-->
-<!--imu link and joint-->
-<!--<link name="imu_link">
-  <inertial>
-    <mass value="1e-5"/>
-    <origin rpy="0 0 0" xyz="0 0 0"/>
-    <inertia ixx="1e-6" ixy="0" ixz="0" iyy="1e-6" iyz="0" izz="1e-6"/>
-  </inertial>
-  <visual>
-    <origin rpy="0 0 0" xyz="0 0 0"/>
-    <geometry>
-      <box size="0.01 0.01 0.01"/>
-    </geometry>
-  </visual>
-  <collision>
-    <origin rpy="0 0 0" xyz="0 0 0"/>
-    <geometry>
-      <box size="0.01 0.01 0.01"/>
-    </geometry>
-  </collision>
-</link>
-<joint name="imu_joint" type="fixed">
-    <origin xyz="0.0.085 0 0.05" rpy= "0 1 0"/>
-    <parent link="link_chassis"/>
-    <child link="imu_link"/>
-    <axis rpy = "0 0 0" xyz="0 1 0"/>
-  </joint>-->
-  <!--imu plugin-->
-  <!--<gazebo reference="imu_link">
-    <sensor name="imu_sensor" type="imu">
-      <always_on>true</always_on>
-      <update_rate>100.0</update_rate>
-      <visualize>true</visualize>
-      <topic>imu_raw</topic>
-      <plugin filename="libgazebo_ros_imu_sensor.so" name="imu_plugin">
-        <topicName>imu/data</topicName>
-        <bodyName>imu_body</bodyName>
-        <updateRateHZ>10.0</updateRateHZ>
-        <gaussianNoise>0.0</gaussianNoise>
-        <xyzOffset>0 0 0</xyzOffset>
-        <rpyOffset>0 0 0</rpyOffset>
-        <frameName>imu_link</frameName>
-        <initialOrientationAsReference>false</initialOrientationAsReference>
-      </plugin>
-    </sensor>
-  </gazebo-->
   <transmission name = "joint_back_left_wheel_trans">
   	<type> transmission_interface/SimpleTransmission </type>

Commit message: 13/04/21 commit

File: src/m2wr_description/urdf/rover.xacro (robot description, xacro)
@@ -297,5 +297,5 @@
   </link>
   <joint name="camera_joint" type="fixed">
-	<origin xyz="0.07 0 0.11" rpy="0 0.5 0"/>
+	<origin xyz="0.08 0 0.11" rpy="0 0.5 0"/>
 	<child link="camera_link"/>
 	<parent link="link_chassis"/>
