Commit message: final edit

File: src/m2wr_description/urdf/rover.xacro (robot description, xacro)
@@ -166,5 +166,5 @@
     <parent link="link_front_right_hinge"/>
     <axis rpy="0 0 0" xyz="0 1 0"/>
-    <limit effort="5" velocity="10"/>
+    <limit effort="5" velocity="22"/>
     <joint_properties damping="0.0" friction="0.0"/>
   </joint>
@@ -174,5 +174,5 @@
     <parent link="link_chassis"/>
     <axis rpy="0 0 0" xyz="0 0 1"/>
-    <limit  effort="5" velocity="5" lower="-0.43" upper="0.33"/>
+    <limit  effort="5" velocity="10" lower="-0.43" upper="0.33"/>
     <joint_properties damping="0.0" friction="0.0"/>
   </joint>
@@ -209,5 +209,5 @@
     <parent link="link_front_left_hinge"/>
     <axis rpy="0 0 0" xyz="0 1 0"/>
-    <limit effort="5" velocity="10"/>
+    <limit effort="5" velocity="22"/>
     <joint_properties damping="0.0" friction="0.0"/>
   </joint>
@@ -217,5 +217,5 @@
     <parent link="link_chassis"/>
     <axis rpy="0 0 0" xyz="0 0 1"/>
-    <limit effort="5" velocity="5" lower= "-0.33" upper="0.44"/>
+    <limit effort="5" velocity="10" lower= "-0.33" upper="0.44"/>
     <joint_properties damping="0.0" friction="0.0"/>
   </joint>
@@ -245,5 +245,5 @@
     <parent link="link_chassis"/>
     <axis rpy="0 0 0" xyz="0 1 0"/>
-    <limit effort="5" velocity="10"/>
+    <limit effort="5" velocity="22"/>
     <joint_properties damping="0.0" friction="0.0"/>
   </joint>
@@ -273,5 +273,5 @@
     <parent link="link_chassis"/>
     <axis rpy="0 0 0" xyz="0 1 0"/>
-    <limit effort="5" velocity="10"/>
+    <limit effort="5" velocity="22"/>
     <joint_properties damping="0.0" friction="0.0"/>
   </joint>
@@ -297,5 +297,5 @@
   </link>
   <joint name="camera_joint" type="fixed">
-	<origin xyz="0.08 0 0.11" rpy="0 0.5 0"/>
+	<origin xyz="0.08 0 0.11" rpy="0 0.55 0"/>
 	<child link="camera_link"/>
 	<parent link="link_chassis"/>
@@ -330,8 +330,8 @@
   	<type> transmission_interface/SimpleTransmission </type>
         <joint name = "joint_back_left_wheel">
-        	<hardwareInterface> hardware_interface/VelocityJointInterface </hardwareInterface>
+        	<hardwareInterface>VelocityJointInterface </hardwareInterface>
         </joint>
         <actuator name = "joint_back_left_wheel_motor">
-                <hardwareInterface> hardware_interface/VelocityJointInterface </hardwareInterface>
+                <hardwareInterface>VelocityJointInterface </hardwareInterface>
   		<mechanicalReduction>1</mechanicalReduction>
 	</actuator>
@@ -340,8 +340,8 @@
   	<type> transmission_interface/SimpleTransmission </type>
         <joint name = "joint_back_right_wheel">
-        	<hardwareInterface> hardware_interface/VelocityJointInterface </hardwareInterface>
+        	<hardwareInterface>VelocityJointInterface </hardwareInterface>
         </joint>
         <actuator name = "joint_back_right_wheel_motor">
-                <hardwareInterface> hardware_interface/VelocityJointInterface </hardwareInterface>
+                <hardwareInterface>VelocityJointInterface </hardwareInterface>
   		<mechanicalReduction>1</mechanicalReduction>
 	</actuator>
@@ -350,8 +350,8 @@
   	<type> transmission_interface/SimpleTransmission </type>
         <joint name = "joint_front_left_hinge">
-        	<hardwareInterface> hardware_interface/PositionJointInterface </hardwareInterface>
+        	<hardwareInterface>PositionJointInterface </hardwareInterface>
         </joint>
         <actuator name = "joint_front_left_hinge_motor">
-                <hardwareInterface> hardware_interface/PositionJointInterface </hardwareInterface>
+                <hardwareInterface>PositionJointInterface </hardwareInterface>
   		<mechanicalReduction>1</mechanicalReduction>
 	</actuator>
@@ -360,8 +360,8 @@
   	<type> transmission_interface/SimpleTransmission </type>
         <joint name = "joint_front_right_hinge">
-        	<hardwareInterface> hardware_interface/PositionJointInterface </hardwareInterface>
+        	<hardwareInterface>PositionJointInterface </hardwareInterface>
         </joint>
         <actuator name = "joint_front_right_hinge_motor">
-                <hardwareInterface> hardware_interface/PositionJointInterface </hardwareInterface>
+                <hardwareInterface>PositionJointInterface </hardwareInterface>
   		<mechanicalReduction>1</mechanicalReduction>
 	</actuator>
@@ -370,4 +370,5 @@
   <plugin name="gazebo_ros_control" filename="libgazebo_ros_control.so">
     <robotNamespace>/rover</robotNamespace>
+    <robotSimType>gazebo_ros_control/DefaultRobotHWSim</robotSimType>
   </plugin>
 </gazebo>
